Commit message: added contact sensor

File: model/robot_core.xacro (robot description, xacro)
@@ -46,4 +46,11 @@
     <gazebo reference="chassis">
         <material>Gazebo/Orange</material>
+        <sensor name="imu_sensor" type="imu">
+            <always_on>1</always_on>
+            <update_rate>100</update_rate>
+            <visualize>true</visualize>
+            <topic>imu</topic>
+            <!-- <pose>0 0 0 0 0 0</pose> -->
+        </sensor>
     </gazebo>
     <!-- LEFT WHEEL LINK -->

File: model/wall.xacro (robot description, xacro)
@@ -1,32 +1,30 @@
 <?xml version="1.0"?>
-<robot xmlns:xacro="http://www.ros.org/wiki/xacro" >
-    <model name='wall'>
-        <static>true</static>
-        <pose>5 0 0 0 0 0</pose><!--pose relative to the world-->
-        <link name='box'>
-            <visual name='visual'>
-                <geometry>
-                    <box>
-                        <size>0.5 10.0 2.0</size>
-                    </box>
-                </geometry>
-                <!--let's add color to our link-->
-                <material>
-                    <ambient>0.0 0.0 1.0 1</ambient>
-                    <diffuse>0.0 0.0 1.0 1</diffuse>
-                    <specular>0.0 0.0 1.0 1</specular>
-                </material>
-            </visual>
-            <collision name='collision'>
-                <geometry>
-                    <box>
-                        <size>0.5 10.0 2.0</size>
-                    </box>
-                </geometry>
-            </collision>
-        </link>
-    </model>
-    <!-- <plugin filename="gz-sim-contact-system"
-            name="gz::sim::systems::Contact">
-    </plugin> -->
+<robot xmlns:xacro="http://www.ros.org/wiki/xacro">
+  <link name="wall">
+    <visual>
+      <origin xyz="5 0 1" rpy="0 0 0"/>
+      <geometry>
+        <box size="0.5 10.0 2.0"/>
+      </geometry>
+      <material name="blue">
+        <color rgba="0.0 0.0 1.0 1"/>
+      </material>
+    </visual>
+    <collision>
+      <origin xyz="5 0 1" rpy="0 0 0"/>
+      <geometry>
+        <box size="0.5 10.0 2.0"/>
+      </geometry>
+    </collision>
+    <inertial>
+      <mass value="1.0"/>
+      <inertia ixx="1.0" iyy="1.0" izz="1.0"
+               ixy="0.0" ixz="0.0" iyz="0.0"/>
+    </inertial>
+  </link>
+  <!-- Tell Gazebo to treat it as static and color it -->
+  <gazebo reference="wall">
+    <static>true</static>
+    <material>Gazebo/Blue</material>
+  </gazebo>
 </robot>
