Commit message: added slam algorithm

File: model/camera.xacro (robot description, xacro)
@@ -47,4 +47,6 @@
             </camera>
             <topic>camera/image_raw</topic>
+            <!-- <always_on>1</always_on> -->
+            <gz_frame_id>camera_link</gz_frame_id>
             <!-- <gz_frame_id>camera_link_optical</gz_frame_id> -->
         </sensor>

File: model/gazebo_control.xacro (robot description, xacro)
@@ -5,6 +5,4 @@
                 name="gz::sim::systems::JointStatePublisher">
                 <topic>/joint_states</topic>
-                <!-- <joint_name>left_wheel_joint</joint_name>
-                <joint_name>right_wheel_joint</joint_name> -->
                 <!-- add any other wheel joints here -->
         </plugin>
@@ -12,11 +10,14 @@
             <left_joint>left_wheel_joint</left_joint>
             <right_joint>right_wheel_joint</right_joint>
+            <topic>/cmd_vel</topic>
+            <odom_topic>/odom</odom_topic>
+            <tf_topic>/tf</tf_topic>
             <wheel_separation>0.297</wheel_separation>
             <wheel_radius>0.05</wheel_radius>
-            <odom_publish_frequency>1</odom_publish_frequency>
-            <topic>cmd_vel</topic>
+            <odom_publish_frequency>100</odom_publish_frequency>
+            <max_acceleration>10.0 10.0</max_acceleration>
+            <child_frame_id>base_link</child_frame_id>
+            <frame_id>odom</frame_id>
         </plugin>
-        <!-- ADD THIS PLUGIN -->
-        <plugin name="gz::sim::systems::JointStatePublisher" filename="gz-sim-joint-state-publisher-system"/>
     </gazebo>
 </robot>

File: model/lidar.xacro (robot description, xacro)
@@ -33,5 +33,5 @@
         <sensor name="laser" type="gpu_lidar">
             <pose> 0 0 0 0 0 0 </pose>
-            <topic>lidar</topic>
+            <topic>/scan</topic>
             <update_rate>10</update_rate>
             <ray>
@@ -58,4 +58,5 @@
             <always_on>1</always_on>
             <visualize>true</visualize>
+            <gz_frame_id>laser_frame</gz_frame_id>
         </sensor>
     </gazebo>

File: model/robot_core.xacro (robot description, xacro)
@@ -19,4 +19,11 @@
     <!-- BASE LINK -->
     <link name="base_link">
+    </link>
+     <joint name="base_footprint_joint" type="fixed">
+        <parent link="base_link"/>
+        <child link="base_footprint"/>
+        <origin xyz="0 0 0" rpy="0 0 0"/>
+    </joint>
+    <link name="base_footprint">
     </link>
     <!-- CHASSIS LINK -->
@@ -50,5 +57,5 @@
             <update_rate>100</update_rate>
             <visualize>true</visualize>
-            <topic>imu</topic>
+            <topic>/imu</topic>
             <!-- <pose>0 0 0 0 0 0</pose> -->
         </sensor>
